Commit message: [dynarm] add version argument and separate urdf and config files

File: robots/v0/dynarm.gazebo.xacro (robot description, xacro)
@@ -4,5 +4,5 @@
   <xacro:arg name="robot_name" default="dynarm" />
   <!-- robot urdf -->
-  <xacro:include filename="$(find dynarm)/robots/dynarm.urdf.xacro" />
+  <xacro:include filename="$(find dynarm)/robots/v0/dynarm.urdf.xacro" />
   <!-- gazebo plugin for default controller and sensors -->
   <xacro:include filename="$(find aerial_robot_simulation)/xacro/spinal.gazebo.xacro" />

File: robots/v0/dynarm.urdf.xacro (robot description, xacro)
@@ -2,7 +2,7 @@
 <robot
     xmlns:xacro="http://www.ros.org/wiki/xacro" name="dynarm" >
-  <xacro:include filename="$(find dynarm)/urdf/common.xacro" />
-  <xacro:include filename="$(find dynarm)/urdf/dynarm_all.xacro" />
-  <xacro:include filename="$(find dynarm)/urdf/gazebo.xacro" />
+  <xacro:include filename="$(find dynarm)/urdf/v0/common.xacro" />
+  <xacro:include filename="$(find dynarm)/urdf/v0/dynarm_all.xacro" />
+  <xacro:include filename="$(find dynarm)/urdf/v0/gazebo.xacro" />
   <!-- root joint -->
   <link name="root">

File: urdf/v0/dynarm_all.xacro (robot description, xacro)
@@ -5,5 +5,5 @@
       <origin xyz="0 0 0" rpy="0 0 0"/>
       <geometry>
-        <mesh filename="package://dynarm/meshes/link0_yaw.STL"/>
+        <mesh filename="package://dynarm/meshes/v0/link0_yaw.STL"/>
       </geometry>
       <material name="">
@@ -21,5 +21,5 @@
       <origin xyz="0 0 0" rpy="0 0 0"/>
       <geometry>
-        <mesh filename="package://dynarm/meshes/link0_pitch.STL"/>
+        <mesh filename="package://dynarm/meshes/v0/link0_pitch.STL"/>
       </geometry>
       <material name="">
@@ -45,5 +45,5 @@
       <origin xyz="0 0 0" rpy="0 0 0"/>
       <geometry>
-        <mesh filename="package://dynarm/meshes/link1.STL"/>
+        <mesh filename="package://dynarm/meshes/v0/link1.STL"/>
       </geometry>
       <material name="">
@@ -69,5 +69,5 @@
       <origin xyz="0 0 0" rpy="0 0 0"/>
       <geometry>
-        <mesh filename="package://dynarm/meshes/joint_junction1.STL"/>
+        <mesh filename="package://dynarm/meshes/v0/joint_junction1.STL"/>
       </geometry>
       <material name="">
@@ -93,5 +93,5 @@
       <origin xyz="0 0 0" rpy="0 0 0"/>
       <geometry>
-        <mesh filename="package://dynarm/meshes/link2.STL"/>
+        <mesh filename="package://dynarm/meshes/v0/link2.STL"/>
       </geometry>
       <material name="">
@@ -117,5 +117,5 @@
       <origin xyz="0 0 0" rpy="0 0 0"/>
       <geometry>
-        <mesh filename="package://dynarm/meshes/joint_junction2.STL"/>
+        <mesh filename="package://dynarm/meshes/v0/joint_junction2.STL"/>
       </geometry>
       <material name="">
@@ -141,5 +141,5 @@
       <origin xyz="0 0 0" rpy="0 0 0"/>
       <geometry>
-        <mesh filename="package://dynarm/meshes/link3.STL"/>
+        <mesh filename="package://dynarm/meshes/v0/link3.STL"/>
       </geometry>
       <material name="">
@@ -165,5 +165,5 @@
       <origin xyz="0 0 0" rpy="0 0 0"/>
       <geometry>
-        <mesh filename="package://dynarm/meshes/joint_junction3.STL"/>
+        <mesh filename="package://dynarm/meshes/v0/joint_junction3.STL"/>
       </geometry>
       <material name="">
@@ -189,5 +189,5 @@
       <origin xyz="0 0 0" rpy="0 0 0"/>
       <geometry>
-        <mesh filename="package://dynarm/meshes/link4.STL"/>
+        <mesh filename="package://dynarm/meshes/v0/link4.STL"/>
       </geometry>
       <material name="">
@@ -213,5 +213,5 @@
       <origin xyz="0 0 0" rpy="0 0 0"/>
       <geometry>
-        <mesh filename="package://dynarm/meshes/gimbal4_roll_link.STL"/>
+        <mesh filename="package://dynarm/meshes/v0/gimbal4_roll_link.STL"/>
       </geometry>
       <material name="">
@@ -237,5 +237,5 @@
       <origin xyz="0 0 0" rpy="0 0 0"/>
       <geometry>
-        <mesh filename="package://dynarm/meshes/gimbal4_pitch_link.STL"/>
+        <mesh filename="package://dynarm/meshes/v0/gimbal4_pitch_link.STL"/>
       </geometry>
       <material name="">
@@ -261,5 +261,5 @@
       <origin xyz="0 0 0" rpy="0 0 0"/>
       <geometry>
-        <mesh filename="package://dynarm/meshes/thrust7.STL"/>
+        <mesh filename="package://dynarm/meshes/v0/thrust7.STL"/>
       </geometry>
       <material name="">
@@ -284,5 +284,5 @@
       <origin xyz="0 0 0" rpy="0 0 0"/>
       <geometry>
-        <mesh filename="package://dynarm/meshes/thrust8.STL"/>
+        <mesh filename="package://dynarm/meshes/v0/thrust8.STL"/>
       </geometry>
       <material name="">
@@ -307,5 +307,5 @@
       <origin xyz="0 0 0" rpy="0 0 0"/>
       <geometry>
-        <mesh filename="package://dynarm/meshes/gimbal3_roll_link.STL"/>
+        <mesh filename="package://dynarm/meshes/v0/gimbal3_roll_link.STL"/>
       </geometry>
       <material name="">
@@ -331,5 +331,5 @@
       <origin xyz="0 0 0" rpy="0 0 0"/>
       <geometry>
-        <mesh filename="package://dynarm/meshes/gimbal3_pitch_link.STL"/>
+        <mesh filename="package://dynarm/meshes/v0/gimbal3_pitch_link.STL"/>
       </geometry>
       <material name="">
@@ -355,5 +355,5 @@
       <origin xyz="0 0 0" rpy="0 0 0"/>
       <geometry>
-        <mesh filename="package://dynarm/meshes/thrust5.STL"/>
+        <mesh filename="package://dynarm/meshes/v0/thrust5.STL"/>
       </geometry>
       <material name="">
@@ -378,5 +378,5 @@
       <origin xyz="0 0 0" rpy="0 0 0"/>
       <geometry>
-        <mesh filename="package://dynarm/meshes/thrust6.STL"/>
+        <mesh filename="package://dynarm/meshes/v0/thrust6.STL"/>
       </geometry>
       <material name="">
@@ -401,5 +401,5 @@
       <origin xyz="0 0 0" rpy="0 0 0"/>
       <geometry>
-        <mesh filename="package://dynarm/meshes/gimbal2_roll_link.STL"/>
+        <mesh filename="package://dynarm/meshes/v0/gimbal2_roll_link.STL"/>
       </geometry>
       <material name="">
@@ -425,5 +425,5 @@
       <origin xyz="0 0 0" rpy="0 0 0"/>
       <geometry>
-        <mesh filename="package://dynarm/meshes/gimbal2_pitch_link.STL"/>
+        <mesh filename="package://dynarm/meshes/v0/gimbal2_pitch_link.STL"/>
       </geometry>
       <material name="">
@@ -449,5 +449,5 @@
       <origin xyz="0 0 0" rpy="0 0 0"/>
       <geometry>
-        <mesh filename="package://dynarm/meshes/thrust3.STL"/>
+        <mesh filename="package://dynarm/meshes/v0/thrust3.STL"/>
       </geometry>
       <material name="">
@@ -472,5 +472,5 @@
       <origin xyz="0 0 0" rpy="0 0 0"/>
       <geometry>
-        <mesh filename="package://dynarm/meshes/thrust4.STL"/>
+        <mesh filename="package://dynarm/meshes/v0/thrust4.STL"/>
       </geometry>
       <material name="">
@@ -495,5 +495,5 @@
       <origin xyz="0 0 0" rpy="0 0 0"/>
       <geometry>
-        <mesh filename="package://dynarm/meshes/gimbal1_roll_link.STL"/>
+        <mesh filename="package://dynarm/meshes/v0/gimbal1_roll_link.STL"/>
       </geometry>
       <material name="">
@@ -519,5 +519,5 @@
       <origin xyz="0 0 0" rpy="0 0 0"/>
       <geometry>
-        <mesh filename="package://dynarm/meshes/gimbal1_pitch_link.STL"/>
+        <mesh filename="package://dynarm/meshes/v0/gimbal1_pitch_link.STL"/>
       </geometry>
       <material name="">
@@ -543,5 +543,5 @@
       <origin xyz="0 0 0" rpy="0 0 0"/>
       <geometry>
-        <mesh filename="package://dynarm/meshes/thrust1.STL"/>
+        <mesh filename="package://dynarm/meshes/v0/thrust1.STL"/>
       </geometry>
       <material name="">
@@ -566,5 +566,5 @@
       <origin xyz="0 0 0" rpy="0 0 0"/>
       <geometry>
-        <mesh filename="package://dynarm/meshes/thrust2.STL"/>
+        <mesh filename="package://dynarm/meshes/v0/thrust2.STL"/>
       </geometry>
       <material name="">
