Commit message: [dynarm][urdf] update v2 urdf. add collision and fix mesh path

File: urdf/v2/dynarm_all.xacro (robot description, xacro)
@@ -5,10 +5,28 @@
       <origin xyz="0 0 0" rpy="0 0 0"/>
       <geometry>
-        <mesh filename="package://dynarm/meshes/link1.STL"/>
-      </geometry>
-      <material name="">
-        <color rgba="0.752941176470588 0.752941176470588 0.752941176470588 1"/>
-      </material>
-    </visual>
+        <mesh filename="package://dynarm/meshes/v2/link1.STL"/>
+      </geometry>
+      <material name="">
+        <color rgba="0.752941176470588 0.752941176470588 0.752941176470588 1"/>
+      </material>
+    </visual>
+    <collision>
+      <origin xyz="0.255 0 0" rpy="0 0 0"/>
+      <geometry>
+        <cylinder length="0.05" radius="0.2"/>
+      </geometry>
+    </collision>
+    <collision>
+      <origin xyz="0.1 0 -0.05" rpy="0 0 0"/>
+      <geometry>
+        <cylinder length="0.1" radius="0.01"/>
+      </geometry>
+    </collision>
+    <collision>
+      <origin xyz="0.41 0 -0.05" rpy="0 0 0"/>
+      <geometry>
+        <cylinder length="0.1" radius="0.01"/>
+      </geometry>
+    </collision>
     <inertial>
       <mass value="0.41284002"/>
@@ -21,5 +39,5 @@
       <origin xyz="0 0 0" rpy="0 0 0"/>
       <geometry>
-        <mesh filename="package://dynarm/meshes/gimbal1_roll_link.STL"/>
+        <mesh filename="package://dynarm/meshes/v2/gimbal1_roll_link.STL"/>
       </geometry>
       <material name="">
@@ -45,10 +63,16 @@
       <origin xyz="0 0 0" rpy="0 0 0"/>
       <geometry>
-        <mesh filename="package://dynarm/meshes/gimbal1_pitch_link.STL"/>
-      </geometry>
-      <material name="">
-        <color rgba="0.752941176470588 0.752941176470588 0.752941176470588 1"/>
-      </material>
-    </visual>
+        <mesh filename="package://dynarm/meshes/v2/gimbal1_pitch_link.STL"/>
+      </geometry>
+      <material name="">
+        <color rgba="0.752941176470588 0.752941176470588 0.752941176470588 1"/>
+      </material>
+    </visual>
+    <collision>
+      <origin xyz="0 0 0" rpy="0 0 0"/>
+      <geometry>
+        <cylinder length="0.05" radius="0.1"/>
+      </geometry>
+    </collision>
     <inertial>
       <mass value="0.46029389"/>
@@ -69,5 +93,5 @@
       <origin xyz="0 0 0" rpy="0 0 0"/>
       <geometry>
-        <mesh filename="package://dynarm/meshes/thrust1.STL"/>
+        <mesh filename="package://dynarm/meshes/v2/thrust1.STL"/>
       </geometry>
       <material name="">
@@ -92,10 +116,16 @@
       <origin xyz="0 0 0" rpy="0 0 0"/>
       <geometry>
-        <mesh filename="package://dynarm/meshes/joint_junction1.STL"/>
-      </geometry>
-      <material name="">
-        <color rgba="0.752941176470588 0.752941176470588 0.752941176470588 1"/>
-      </material>
-    </visual>
+        <mesh filename="package://dynarm/meshes/v2/joint_junction1.STL"/>
+      </geometry>
+      <material name="">
+        <color rgba="0.752941176470588 0.752941176470588 0.752941176470588 1"/>
+      </material>
+    </visual>
+    <collision>
+      <origin xyz="0.0835 0 0" rpy="0 0 0"/>
+      <geometry>
+        <box size="0.167 0.05 0.05"/>
+      </geometry>
+    </collision>
     <inertial>
       <mass value="0.77592368"/>
@@ -116,10 +146,28 @@
       <origin xyz="0 0 0" rpy="0 0 0"/>
       <geometry>
-        <mesh filename="package://dynarm/meshes/link2.STL"/>
-      </geometry>
-      <material name="">
-        <color rgba="0.752941176470588 0.752941176470588 0.752941176470588 1"/>
-      </material>
-    </visual>
+        <mesh filename="package://dynarm/meshes/v2/link2.STL"/>
+      </geometry>
+      <material name="">
+        <color rgba="0.752941176470588 0.752941176470588 0.752941176470588 1"/>
+      </material>
+    </visual>
+    <collision>
+      <origin xyz="0.24 0 0" rpy="0 0 0"/>
+      <geometry>
+        <cylinder length="0.05" radius="0.2"/>
+      </geometry>
+    </collision>
+    <collision>
+      <origin xyz="0.085 0 -0.05" rpy="0 0 0"/>
+      <geometry>
+        <cylinder length="0.1" radius="0.01"/>
+      </geometry>
+    </collision>
+    <collision>
+      <origin xyz="0.395 0 -0.05" rpy="0 0 0"/>
+      <geometry>
+        <cylinder length="0.1" radius="0.01"/>
+      </geometry>
+    </collision>
     <inertial>
       <mass value="0.44741891"/>
@@ -140,5 +188,5 @@
       <origin xyz="0 0 0" rpy="0 0 0"/>
       <geometry>
-        <mesh filename="package://dynarm/meshes/gimbal2_roll_link.STL"/>
+        <mesh filename="package://dynarm/meshes/v2/gimbal2_roll_link.STL"/>
       </geometry>
       <material name="">
@@ -164,10 +212,16 @@
       <origin xyz="0 0 0" rpy="0 0 0"/>
       <geometry>
-        <mesh filename="package://dynarm/meshes/gimbal2_pitch_link.STL"/>
-      </geometry>
-      <material name="">
-        <color rgba="0.752941176470588 0.752941176470588 0.752941176470588 1"/>
-      </material>
-    </visual>
+        <mesh filename="package://dynarm/meshes/v2/gimbal2_pitch_link.STL"/>
+      </geometry>
+      <material name="">
+        <color rgba="0.752941176470588 0.752941176470588 0.752941176470588 1"/>
+      </material>
+    </visual>
+    <collision>
+      <origin xyz="0 0 0" rpy="0 0 0"/>
+      <geometry>
+        <cylinder length="0.05" radius="0.1"/>
+      </geometry>
+    </collision>
     <inertial>
       <mass value="0.46029389"/>
@@ -188,5 +242,5 @@
       <origin xyz="0 0 0" rpy="0 0 0"/>
       <geometry>
-        <mesh filename="package://dynarm/meshes/thrust2.STL"/>
+        <mesh filename="package://dynarm/meshes/v2/thrust2.STL"/>
       </geometry>
       <material name="">
@@ -211,10 +265,16 @@
       <origin xyz="0 0 0" rpy="0 0 0"/>
       <geometry>
-        <mesh filename="package://dynarm/meshes/joint_junction2.STL"/>
-      </geometry>
-      <material name="">
-        <color rgba="0.752941176470588 0.752941176470588 0.752941176470588 1"/>
-      </material>
-    </visual>
+        <mesh filename="package://dynarm/meshes/v2/joint_junction2.STL"/>
+      </geometry>
+      <material name="">
+        <color rgba="0.752941176470588 0.752941176470588 0.752941176470588 1"/>
+      </material>
+    </visual>
+    <collision>
+      <origin xyz="0.0835 0 0" rpy="0 0 0"/>
+      <geometry>
+        <box size="0.167 0.05 0.05"/>
+      </geometry>
+    </collision>
     <inertial>
       <mass value="0.77592368"/>
@@ -235,10 +295,28 @@
       <origin xyz="0 0 0" rpy="0 0 0"/>
       <geometry>
-        <mesh filename="package://dynarm/meshes/link3.STL"/>
-      </geometry>
-      <material name="">
-        <color rgba="0.752941176470588 0.752941176470588 0.752941176470588 1"/>
-      </material>
-    </visual>
+        <mesh filename="package://dynarm/meshes/v2/link3.STL"/>
+      </geometry>
+      <material name="">
+        <color rgba="0.752941176470588 0.752941176470588 0.752941176470588 1"/>
+      </material>
+    </visual>
+    <collision>
+      <origin xyz="0.24 0 0" rpy="0 0 0"/>
+      <geometry>
+        <cylinder length="0.05" radius="0.2"/>
+      </geometry>
+    </collision>
+    <collision>
+      <origin xyz="0.085 0 -0.05" rpy="0 0 0"/>
+      <geometry>
+        <cylinder length="0.1" radius="0.01"/>
+      </geometry>
+    </collision>
+    <collision>
+      <origin xyz="0.395 0 -0.05" rpy="0 0 0"/>
+      <geometry>
+        <cylinder length="0.1" radius="0.01"/>
+      </geometry>
+    </collision>
     <inertial>
       <mass value="0.44741891"/>
@@ -259,5 +337,5 @@
       <origin xyz="0 0 0" rpy="0 0 0"/>
       <geometry>
-        <mesh filename="package://dynarm/meshes/gimbal3_roll_link.STL"/>
+        <mesh filename="package://dynarm/meshes/v2/gimbal3_roll_link.STL"/>
       </geometry>
       <material name="">
@@ -283,10 +361,16 @@
       <origin xyz="0 0 0" rpy="0 0 0"/>
       <geometry>
-        <mesh filename="package://dynarm/meshes/gimbal3_pitch_link.STL"/>
-      </geometry>
-      <material name="">
-        <color rgba="0.752941176470588 0.752941176470588 0.752941176470588 1"/>
-      </material>
-    </visual>
+        <mesh filename="package://dynarm/meshes/v2/gimbal3_pitch_link.STL"/>
+      </geometry>
+      <material name="">
+        <color rgba="0.752941176470588 0.752941176470588 0.752941176470588 1"/>
+      </material>
+    </visual>
+    <collision>
+      <origin xyz="0 0 0" rpy="0 0 0"/>
+      <geometry>
+        <cylinder length="0.05" radius="0.1"/>
+      </geometry>
+    </collision>
     <inertial>
       <mass value="0.46029389"/>
@@ -307,5 +391,5 @@
       <origin xyz="0 0 0" rpy="0 0 0"/>
       <geometry>
-        <mesh filename="package://dynarm/meshes/thrust3.STL"/>
+        <mesh filename="package://dynarm/meshes/v2/thrust3.STL"/>
       </geometry>
       <material name="">
@@ -330,10 +414,16 @@
       <origin xyz="0 0 0" rpy="0 0 0"/>
       <geometry>
-        <mesh filename="package://dynarm/meshes/joint_junction3.STL"/>
-      </geometry>
-      <material name="">
-        <color rgba="0.752941176470588 0.752941176470588 0.752941176470588 1"/>
-      </material>
-    </visual>
+        <mesh filename="package://dynarm/meshes/v2/joint_junction3.STL"/>
+      </geometry>
+      <material name="">
+        <color rgba="0.752941176470588 0.752941176470588 0.752941176470588 1"/>
+      </material>
+    </visual>
+    <collision>
+      <origin xyz="0.0835 0 0" rpy="0 0 0"/>
+      <geometry>
+        <box size="0.167 0.05 0.05"/>
+      </geometry>
+    </collision>
     <inertial>
       <mass value="0.77592368"/>
@@ -354,10 +444,28 @@
       <origin xyz="0 0 0" rpy="0 0 0"/>
       <geometry>
-        <mesh filename="package://dynarm/meshes/link4.STL"/>
-      </geometry>
-      <material name="">
-        <color rgba="0.752941176470588 0.752941176470588 0.752941176470588 1"/>
-      </material>
-    </visual>
+        <mesh filename="package://dynarm/meshes/v2/link4.STL"/>
+      </geometry>
+      <material name="">
+        <color rgba="0.752941176470588 0.752941176470588 0.752941176470588 1"/>
+      </material>
+    </visual>
+    <collision>
+      <origin xyz="0.24 0 0" rpy="0 0 0"/>
+      <geometry>
+        <cylinder length="0.05" radius="0.2"/>
+      </geometry>
+    </collision>
+    <collision>
+      <origin xyz="0.085 0 -0.05" rpy="0 0 0"/>
+      <geometry>
+        <cylinder length="0.1" radius="0.01"/>
+      </geometry>
+    </collision>
+    <collision>
+      <origin xyz="0.395 0 -0.05" rpy="0 0 0"/>
+      <geometry>
+        <cylinder length="0.1" radius="0.01"/>
+      </geometry>
+    </collision>
     <inertial>
       <mass value="0.41284002"/>
@@ -378,5 +486,5 @@
       <origin xyz="0 0 0" rpy="0 0 0"/>
       <geometry>
-        <mesh filename="package://dynarm/meshes/gimbal4_roll_link.STL"/>
+        <mesh filename="package://dynarm/meshes/v2/gimbal4_roll_link.STL"/>
       </geometry>
       <material name="">
@@ -402,10 +510,16 @@
       <origin xyz="0 0 0" rpy="0 0 0"/>
       <geometry>
-        <mesh filename="package://dynarm/meshes/gimbal4_pitch_link.STL"/>
-      </geometry>
-      <material name="">
-        <color rgba="0.752941176470588 0.752941176470588 0.752941176470588 1"/>
-      </material>
-    </visual>
+        <mesh filename="package://dynarm/meshes/v2/gimbal4_pitch_link.STL"/>
+      </geometry>
+      <material name="">
+        <color rgba="0.752941176470588 0.752941176470588 0.752941176470588 1"/>
+      </material>
+    </visual>
+    <collision>
+      <origin xyz="0 0 0" rpy="0 0 0"/>
+      <geometry>
+        <cylinder length="0.05" radius="0.1"/>
+      </geometry>
+    </collision>
     <inertial>
       <mass value="0.46029389"/>
@@ -426,5 +540,5 @@
       <origin xyz="0 0 0" rpy="0 0 0"/>
       <geometry>
-        <mesh filename="package://dynarm/meshes/thrust4.STL"/>
+        <mesh filename="package://dynarm/meshes/v2/thrust4.STL"/>
       </geometry>
       <material name="">
