Commit message: [dynarm][urdf] fix data about max thrust

File: urdf/v1/dynarm_all.xacro (robot description, xacro)
@@ -134,5 +134,5 @@
     <child link="thrust1"/>
     <axis xyz="0 0 1"/>
-    <limit lower="0.0" upper="25.0" effort="100" velocity="0.5"/>
+    <limit lower="0.0" upper="38.0" effort="100" velocity="0.5"/>
   </joint>
   <link name="joint_junction1">
@@ -253,5 +253,5 @@
     <child link="thrust2"/>
     <axis xyz="0 0 -1"/>
-    <limit lower="0.0" upper="25.0" effort="100" velocity="0.5"/>
+    <limit lower="0.0" upper="38.0" effort="100" velocity="0.5"/>
   </joint>
   <link name="joint_junction2">
@@ -372,5 +372,5 @@
     <child link="thrust3"/>
     <axis xyz="0 0 1"/>
-    <limit lower="0.0" upper="25.0" effort="100" velocity="0.5"/>
+    <limit lower="0.0" upper="38.0" effort="100" velocity="0.5"/>
   </joint>
 </robot>

Commit message: [dynarm][urdf] add collision and friction to urdf

File: urdf/v1/dynarm_all.xacro (robot description, xacro)
@@ -11,4 +11,10 @@
       </material>
     </visual>
+    <collision>
+      <origin xyz="0.025 0 0" rpy="0 ${pi / 2} 0"/>
+      <geometry>
+        <cylinder length="0.05" radius="0.05"/>
+      </geometry>
+    </collision>
     <inertial>
       <mass value="1.0761005"/>
@@ -27,4 +33,10 @@
       </material>
     </visual>
+    <collision>
+      <origin xyz="0.062 0 0" rpy="${pi / 2} 0 0"/>
+      <geometry>
+        <cylinder length="0.05" radius="0.05"/>
+      </geometry>
+    </collision>
     <inertial>
       <mass value="1.24295185"/>
@@ -51,4 +63,22 @@
       </material>
     </visual>
+    <collision>
+      <origin xyz="0.292 0 0" rpy="0 0 0"/>
+      <geometry>
+        <cylinder length="0.05" radius="0.2"/>
+      </geometry>
+    </collision>
+    <collision>
+      <origin xyz="0.137 0 -0.05" rpy="0 0 0"/>
+      <geometry>
+        <cylinder length="0.1" radius="0.01"/>
+      </geometry>
+    </collision>
+    <collision>
+      <origin xyz="0.447 0 -0.05" rpy="0 0 0"/>
+      <geometry>
+        <cylinder length="0.1" radius="0.01"/>
+      </geometry>
+    </collision>
     <inertial>
       <mass value="0.56565523"/>
@@ -99,4 +129,10 @@
       </material>
     </visual>
+    <collision>
+      <origin xyz="0 0 0" rpy="0 0 0"/>
+      <geometry>
+        <cylinder length="0.05" radius="0.1"/>
+      </geometry>
+    </collision>
     <inertial>
       <mass value="0.45023026"/>
@@ -146,4 +182,10 @@
       </material>
     </visual>
+    <collision>
+      <origin xyz="0.0835 0 0" rpy="0 0 0"/>
+      <geometry>
+        <box size="0.167 0.05 0.05"/>
+      </geometry>
+    </collision>
     <inertial>
       <mass value="0.77591975"/>
@@ -170,4 +212,22 @@
       </material>
     </visual>
+    <collision>
+      <origin xyz="0.24 0 0" rpy="0 0 0"/>
+      <geometry>
+        <cylinder length="0.05" radius="0.2"/>
+      </geometry>
+    </collision>
+    <collision>
+      <origin xyz="0.085 0 -0.05" rpy="0 0 0"/>
+      <geometry>
+        <cylinder length="0.1" radius="0.01"/>
+      </geometry>
+    </collision>
+    <collision>
+      <origin xyz="0.395 0 -0.05" rpy="0 0 0"/>
+      <geometry>
+        <cylinder length="0.1" radius="0.01"/>
+      </geometry>
+    </collision>
     <inertial>
       <mass value="0.44767426"/>
@@ -218,4 +278,10 @@
       </material>
     </visual>
+    <collision>
+      <origin xyz="0 0 0" rpy="0 0 0"/>
+      <geometry>
+        <cylinder length="0.05" radius="0.1"/>
+      </geometry>
+    </collision>
     <inertial>
       <mass value="0.45023026"/>
@@ -265,4 +331,10 @@
       </material>
     </visual>
+    <collision>
+      <origin xyz="0.0835 0 0" rpy="0 0 0"/>
+      <geometry>
+        <box size="0.167 0.05 0.05"/>
+      </geometry>
+    </collision>
     <inertial>
       <mass value="0.77591975"/>
@@ -289,4 +361,22 @@
       </material>
     </visual>
+    <collision>
+      <origin xyz="0.24 0 0" rpy="0 0 0"/>
+      <geometry>
+        <cylinder length="0.05" radius="0.2"/>
+      </geometry>
+    </collision>
+    <collision>
+      <origin xyz="0.085 0 -0.05" rpy="0 0 0"/>
+      <geometry>
+        <cylinder length="0.1" radius="0.01"/>
+      </geometry>
+    </collision>
+    <collision>
+      <origin xyz="0.395 0 -0.05" rpy="0 0 0"/>
+      <geometry>
+        <cylinder length="0.1" radius="0.01"/>
+      </geometry>
+    </collision>
     <inertial>
       <mass value="0.41309537"/>
@@ -337,4 +427,10 @@
       </material>
     </visual>
+    <collision>
+      <origin xyz="0 0 0" rpy="0 0 0"/>
+      <geometry>
+        <cylinder length="0.05" radius="0.1"/>
+      </geometry>
+    </collision>
     <inertial>
       <mass value="0.45023026"/>

File: urdf/v1/gazebo.xacro (robot description, xacro)
@@ -151,3 +151,16 @@
     </actuator>
   </transmission>
+  <!-- friction -->
+  <gazebo reference="link1">
+    <mu1>0.4</mu1>
+    <mu2>0.4</mu2>
+  </gazebo>
+  <gazebo reference="link2">
+    <mu1>0.4</mu1>
+    <mu2>0.4</mu2>
+  </gazebo>
+  <gazebo reference="link3">
+    <mu1>0.4</mu1>
+    <mu2>0.4</mu2>
+  </gazebo>
 </robot>

Commit message: [v1][urdf] update thrust limits

File: urdf/v1/dynarm_all.xacro (robot description, xacro)
@@ -170,5 +170,5 @@
     <child link="thrust1"/>
     <axis xyz="0 0 1"/>
-    <limit lower="0.0" upper="38.0" effort="100" velocity="0.5"/>
+    <limit lower="7.1" upper="40.0" effort="100" velocity="0.5"/>
   </joint>
   <link name="joint_junction1">
@@ -319,5 +319,5 @@
     <child link="thrust2"/>
     <axis xyz="0 0 -1"/>
-    <limit lower="0.0" upper="38.0" effort="100" velocity="0.5"/>
+    <limit lower="7.1" upper="40.0" effort="100" velocity="0.5"/>
   </joint>
   <link name="joint_junction2">
@@ -468,5 +468,5 @@
     <child link="thrust3"/>
     <axis xyz="0 0 1"/>
-    <limit lower="0.0" upper="38.0" effort="100" velocity="0.5"/>
+    <limit lower="7.1" upper="40.0" effort="100" velocity="0.5"/>
   </joint>
 </robot>
