Commit message: change gazebo visual to stl

File: urdf/v3/dynarm_all.xacro (robot description, xacro)
@@ -9,5 +9,5 @@
     <visual>
       <geometry>
-        <mesh filename="package://dynarm/meshes/v3/base_link.dae"/>
+        <mesh filename="package://dynarm/meshes/v3/base_link.stl"/>
       </geometry>
       <material name="__unnamed_material_1"/>
@@ -23,5 +23,5 @@
     <visual>
       <geometry>
-        <mesh filename="package://dynarm/meshes/v3/link1.dae"/>
+        <mesh filename="package://dynarm/meshes/v3/link1.stl"/>
       </geometry>
       <material name="__unnamed_material_2"/>
@@ -37,5 +37,5 @@
     <visual>
       <geometry>
-        <mesh filename="package://dynarm/meshes/v3/gimbal1_roll_link.dae"/>
+        <mesh filename="package://dynarm/meshes/v3/gimbal1_roll_link.stl"/>
       </geometry>
       <material name="__unnamed_material_3"/>
@@ -51,5 +51,5 @@
     <visual>
       <geometry>
-        <mesh filename="package://dynarm/meshes/v3/gimbal1_pitch_link.dae"/>
+        <mesh filename="package://dynarm/meshes/v3/gimbal1_pitch_link.stl"/>
       </geometry>
       <material name="__unnamed_material_4"/>
@@ -65,5 +65,5 @@
     <visual>
       <geometry>
-        <mesh filename="package://dynarm/meshes/v3/thrust1.dae"/>
+        <mesh filename="package://dynarm/meshes/v3/thrust1.stl"/>
       </geometry>
       <material name="__unnamed_material_5"/>
@@ -79,5 +79,5 @@
     <visual>
       <geometry>
-        <mesh filename="package://dynarm/meshes/v3/link2.dae"/>
+        <mesh filename="package://dynarm/meshes/v3/link2.stl"/>
       </geometry>
       <material name="__unnamed_material_6"/>
@@ -93,5 +93,5 @@
     <visual>
       <geometry>
-        <mesh filename="package://dynarm/meshes/v3/gimbal2_roll_link.dae"/>
+        <mesh filename="package://dynarm/meshes/v3/gimbal2_roll_link.stl"/>
       </geometry>
       <material name="__unnamed_material_7"/>
@@ -107,5 +107,5 @@
     <visual>
       <geometry>
-        <mesh filename="package://dynarm/meshes/v3/gimbal2_pitch_link.dae"/>
+        <mesh filename="package://dynarm/meshes/v3/gimbal2_pitch_link.stl"/>
       </geometry>
       <material name="__unnamed_material_8"/>
@@ -121,5 +121,5 @@
     <visual>
       <geometry>
-        <mesh filename="package://dynarm/meshes/v3/thrust2.dae"/>
+        <mesh filename="package://dynarm/meshes/v3/thrust2.stl"/>
       </geometry>
       <material name="__unnamed_material_9"/>
@@ -135,5 +135,5 @@
     <visual>
       <geometry>
-        <mesh filename="package://dynarm/meshes/v3/link3.dae"/>
+        <mesh filename="package://dynarm/meshes/v3/link3.stl"/>
       </geometry>
       <material name="__unnamed_material_10"/>
