Commit message: fix typo in macro

File: urdf/v3/common.xacro (robot description, xacro)
@@ -18,5 +18,5 @@
   <!-- macro of virtual link -->
   <xacro:macro name="virtual_link" params="parent child xyz:='0 0 0' rpy:='0 0 0'">
-    <link name="child"/>
+    <link name="${child}"/>
     <joint name="${parent}_2_${child}" type="fixed">
       <parent link="${parent}"/>
