Commit message: update urdf

File: robots/v3/dynarm.gazebo.xacro (robot description, xacro)
@@ -18,3 +18,7 @@
   <xacro:rotor_transmission id="1"/>
   <xacro:rotor_transmission id="2"/>
+  <!-- friction -->
+  <xacro:gazebo_friction link="link1"/>
+  <xacro:gazebo_friction link="link2"/>
+  <xacro:gazebo_friction link="link3"/>
 </robot>

File: urdf/v3/common.xacro (robot description, xacro)
@@ -50,3 +50,10 @@
     </transmission>
   </xacro:macro>
+  <!-- friction -->
+  <xacro:macro name="gazebo_friction" params="link">
+    <gazebo reference="${link}">
+      <mu1>0.4</mu1>
+      <mu2>0.4</mu2>
+    </gazebo>
+  </xacro:macro>
 </robot>

File: urdf/v3/dynarm_all.xacro (robot description, xacro)
@@ -3,7 +3,7 @@
   <link name="base_link">
     <inertial>
-      <origin xyz="0.027111559582523 0.00165632549449175 1.3437401002616e-09" rpy="0.0 -0.0 0.0"/>
-      <mass value="0.490000522187397"/>
-      <inertia ixx="0.000198107312535685" ixy="-6.96972575146703e-07" ixz="6.50710842999406e-08" iyy="0.000213284145580095" iyz="-1.01698023263196e-11" izz="0.000189175868864902"/>
+      <origin xyz="0.02670275 0.00180026 0.00000000" rpy="0 0 0"/>
+      <mass value="0.45218521"/>
+      <inertia ixx="0.00035567" ixy="-0.00000519" ixz="-0.00000005" iyy="0.00023609" iyz="0.00000000" izz="0.00038211"/>
     </inertial>
     <visual>
@@ -17,7 +17,7 @@
   <link name="link1">
     <inertial>
-      <origin xyz="0.3459227611967 -0.000221078938689229 0.0153188536699517" rpy="0.0 -0.0 0.0"/>
-      <mass value="1.85632504317605"/>
-      <inertia ixx="0.0108448412120977" ixy="-5.6416499725003e-07" ixz="2.96991333310925e-07" iyy="0.0156637188549782" iyz="5.88810884503775e-08" izz="0.024018838204809"/>
+      <origin xyz="0.35205652 -0.00007679 0.02097532" rpy="0 0 0"/>
+      <mass value="1.36722322"/>
+      <inertia ixx="0.01379981" ixy="0.00032493" ixz="-0.00158041" iyy="0.05561425" iyz="-0.00001203" izz="0.05909683"/>
     </inertial>
     <visual>
@@ -31,7 +31,7 @@
   <link name="gimbal1_roll_link">
     <inertial>
-      <origin xyz="-0.00783546366619609 -0.0324699030903514 1.64826370592793e-06" rpy="0.0 -0.0 0.0"/>
-      <mass value="0.29135232532025"/>
-      <inertia ixx="0.00161603335066671" ixy="9.08174410370115e-07" ixz="4.40820031639382e-09" iyy="0.000344744394264198" iyz="5.23305789314138e-09" izz="0.00188868729102949"/>
+      <origin xyz="-0.01041514 -0.03581395 0.00000195" rpy="0 0 0"/>
+      <mass value="0.31718547"/>
+      <inertia ixx="0.00322436" ixy="-0.00001817" ixz="0.00000000" iyy="0.00357664" iyz="-0.00000008" izz="0.00671390"/>
     </inertial>
     <visual>
@@ -45,7 +45,7 @@
   <link name="gimbal1_pitch_link">
     <inertial>
-      <origin xyz="-6.99171337977811e-05 -0.000443866346860996 0.00162824501615241" rpy="0.0 -0.0 0.0"/>
-      <mass value="0.409711618848904"/>
-      <inertia ixx="0.00125969767885536" ixy="6.17380392220277e-07" ixz="-5.03873537223111e-07" iyy="0.00103671312020798" iyz="1.25621062897587e-05" izz="0.00202112119538432"/>
+      <origin xyz="-0.00008734 -0.00066322 0.00149887" rpy="0 0 0"/>
+      <mass value="0.42303791"/>
+      <inertia ixx="0.00176884" ixy="-0.00000081" ixz="0.00000078" iyy="0.00088469" iyz="-0.00000058" izz="0.00236242"/>
     </inertial>
     <visual>
@@ -58,9 +58,5 @@
   </link>
   <link name="thrust1">
-    <inertial>
-      <origin xyz="1.08136435422734e-06 -5.59005514422567e-07 0.00395854941642201" rpy="0.0 -0.0 0.0"/>
-      <mass value="0.0107232111514425"/>
-      <inertia ixx="1.65582387978783e-05" ixy="2.64405902452945e-10" ixz="-6.36535202066436e-11" iyy="1.65577469248177e-05" iyz="-8.56721496798493e-12" izz="3.3077650948732e-05"/>
-    </inertial>
+    <xacro:virtual_inertial/>
     <visual>
       <geometry>
@@ -73,7 +69,7 @@
   <link name="link2">
     <inertial>
-      <origin xyz="0.345922761187255 -0.000221078932155115 0.0153188536674012" rpy="0.0 -0.0 0.0"/>
-      <mass value="1.8563250433674"/>
-      <inertia ixx="0.0108448412121155" ixy="-5.64164996967007e-07" ixz="2.96991332357008e-07" iyy="0.0156637188549864" iyz="5.88810875578539e-08" izz="0.0240188382048185"/>
+      <origin xyz="0.35205652 -0.00007679 0.02097532" rpy="0 0 0"/>
+      <mass value="1.36722322"/>
+      <inertia ixx="0.01379981" ixy="0.00032493" ixz="-0.00158041" iyy="0.05561425" iyz="-0.00001203" izz="0.05909683"/>
     </inertial>
     <visual>
@@ -87,7 +83,7 @@
   <link name="gimbal2_roll_link">
     <inertial>
-      <origin xyz="-0.00783546360767251 -0.0324699030947344 1.64831496667882e-06" rpy="0.0 -0.0 0.0"/>
-      <mass value="0.291352325353693"/>
-      <inertia ixx="0.00161603335066697" ixy="9.08174410696797e-07" ixz="4.40820023795866e-09" iyy="0.00034474439426527" iyz="5.23305784752353e-09" izz="0.00188868729103088"/>
+      <origin xyz="-0.01041514 -0.03581395 0.00000195" rpy="0 0 0"/>
+      <mass value="0.31718547"/>
+      <inertia ixx="0.00322436" ixy="-0.00001817" ixz="0.00000000" iyy="0.00357664" iyz="-0.00000008" izz="0.00671390"/>
     </inertial>
     <visual>
@@ -101,7 +97,7 @@
   <link name="gimbal2_pitch_link">
     <inertial>
-      <origin xyz="-6.99171338204296e-05 -0.000443866346266648 0.00162824501608197" rpy="0.0 -0.0 0.0"/>
-      <mass value="0.409711618847066"/>
-      <inertia ixx="0.00125969767885561" ixy="6.17380392191852e-07" ixz="-5.03873537220234e-07" iyy="0.00103671312020799" iyz="1.25621062897626e-05" izz="0.00202112119538455"/>
+      <origin xyz="-0.00008734 -0.00066322 0.00149887" rpy="0 0 0"/>
+      <mass value="0.42303791"/>
+      <inertia ixx="0.00176884" ixy="-0.00000081" ixz="0.00000078" iyy="0.00088469" iyz="-0.00000058" izz="0.00236242"/>
     </inertial>
     <visual>
@@ -114,9 +110,5 @@
   </link>
   <link name="thrust2">
-    <inertial>
-      <origin xyz="9.08944965405389e-07 -6.38348894601007e-07 0.00395854992447526" rpy="0.0 -0.0 0.0"/>
-      <mass value="0.0107232454039342"/>
-      <inertia ixx="1.65582691015053e-05" ixy="2.03708555861106e-10" ixz="-6.38647659964995e-11" iyy="1.65578719942898e-05" iyz="-8.85544756614096e-12" izz="3.30778062428382e-05"/>
-    </inertial>
+    <xacro:virtual_inertial/>
     <visual>
       <geometry>
@@ -129,7 +121,7 @@
   <link name="link3">
     <inertial>
-      <origin xyz="0.0582149613585146 -0.00176173194949543 3.8361490812658e-09" rpy="0.0 -0.0 0.0"/>
-      <mass value="0.105760535828491"/>
-      <inertia ixx="1.36775986135056e-05" ixy="-1.71368753621589e-08" ixz="4.16604448211742e-12" iyy="0.000105563860087045" iyz="-7.45684977109264e-12" izz="0.00010330461617006"/>
+      <origin xyz="0.05896281 -0.00153878 0.00000000" rpy="0 0 0"/>
+      <mass value="0.10242647"/>
+      <inertia ixx="0.00004853" ixy="0.00001138" ixz="0.00000000" iyy="0.00033848" iyz="0.00000000" izz="0.00036698"/>
     </inertial>
     <visual>
@@ -147,4 +139,5 @@
     <axis xyz="0. 1. 0."/>
     <origin xyz="0.032 0.0 0.0" rpy="0.0 -0.0 0.0"/>
+    <dynamics damping="0.9" friction="0.7"/>
   </joint>
   <joint name="gimbal1_roll" type="revolute">
@@ -154,4 +147,5 @@
     <axis xyz="1. 0. 0."/>
     <origin xyz="0.2885 0.0 0.0" rpy="0.0 -0.0 0.0"/>
+    <dynamics damping="0.1" friction="0.0"/>
   </joint>
   <joint name="gimbal1_pitch" type="revolute">
@@ -161,4 +155,5 @@
     <axis xyz="0. 1. 0."/>
     <origin xyz="0.0 0.0 0.0" rpy="0.0 -0.0 0.0"/>
+    <dynamics damping="0.1" friction="0.0"/>
   </joint>
   <joint name="rotor1" type="continuous">
@@ -175,4 +170,5 @@
     <axis xyz="0. 1. 0."/>
     <origin xyz="0.577 0.0 0.0" rpy="0.0 -0.0 0.0"/>
+    <dynamics damping="0.9" friction="0.7"/>
   </joint>
   <joint name="gimbal2_roll" type="revolute">
@@ -182,4 +178,5 @@
     <axis xyz="1. 0. 0."/>
     <origin xyz="0.2885 0.0 0.0" rpy="0.0 -0.0 0.0"/>
+    <dynamics damping="0.1" friction="0.0"/>
   </joint>
   <joint name="gimbal2_pitch" type="revolute">
@@ -189,4 +186,5 @@
     <axis xyz="0. 1. 0."/>
     <origin xyz="0.0 0.0 0.0" rpy="0.0 -0.0 0.0"/>
+    <dynamics damping="0.1" friction="0.0"/>
   </joint>
   <joint name="rotor2" type="continuous">
@@ -203,4 +201,5 @@
     <axis xyz="0. 1. 0."/>
     <origin xyz="0.577 0.0 0.0" rpy="0.0 -0.0 0.0"/>
+    <dynamics damping="0.9" friction="0.7"/>
   </joint>
   <material name="__unnamed_material_1">
